Commit message: [FEAT] Add camera and LIDAR

File: catkin_ws/src/go_chase_it/urdf/my_robot.xacro (robot description, xacro)
@@ -78,5 +78,5 @@
      </inertial>
   </link>
- <link name= 'right_wheel'>
+  <link name= 'right_wheel'>
     <visual>
       <origin xyz="-0.0 0 0" rpy=" 0 1.5707 1.5707"/>
@@ -101,4 +101,62 @@
     </inertial>
   </link>
+  <link name='camera'>
+    <visual>
+      <origin xyz="-0.0 0 0" rpy=" 0 0 0"/>
+      <geometry>
+        <box size="0.05 0.05 0.05"/>
+      </geometry>
+    </visual>
+     <collision>
+      <origin xyz="-0.0 0 0" rpy=" 0 0 0"/>
+      <geometry>
+        <box size="0.05 0.05 0.05"/>
+      </geometry>
+    </collision>
+    <inertial>
+      <mass value="0.1"/>
+      <origin xyz="0.0 0 0" rpy=" 0 0 0"/>
+      <inertia
+          ixx="1e-6" ixy="0" ixz="0"
+          iyy="1e-6" iyz="0"
+          izz="1e-6"
+      />
+    </inertial>
+  </link>
+<link name='hokuyo'>
+    <visual>
+      <origin xyz="-0.0 0 0" rpy=" 0 0 0"/>
+      <geometry>
+        <mesh filename="package://go_chase_it/meshes/hokuyo.dae"/>
+      </geometry>
+    </visual>
+    <collision>
+      <origin xyz="-0.0 0 0" rpy=" 0 0 0"/>
+      <geometry>
+        <box size="0.01 0.01 0.01"/>
+      </geometry>
+    </collision>
+    <inertial>
+      <mass value="1e-5"/>
+      <origin xyz="0.0 0 0" rpy=" 0 0 0"/>
+      <inertia
+          ixx="1e-6" ixy="0" ixz="0"
+          iyy="1e-6" iyz="0"
+          izz="1e-6"
+      />
+    </inertial>
+  </link>
+  <joint type="fixed" name="camera_joint">
+    <origin xyz="0.2 0 0" rpy="0 0 0"/>
+    <child link="camera"/>
+    <parent link="chassis"/>
+    <axis xyz="0 1 0" rpy="0 0 0"/>
+  </joint>
+  <joint type="fixed" name="hokuyo">
+    <origin xyz="0.15 0 0.1" rpy="0 0 0"/>
+    <child link="hokuyo"/>
+    <parent link="chassis"/>
+    <axis xyz="0 1 0" rpy="0 0 0"/>
+  </joint>
   <joint type="continuous" name="left_wheel_hinge">
     <origin xyz="0 0.15 0" rpy="0 0 0"/>
@@ -108,6 +166,6 @@
     <limit effort="10000" velocity="1000"/>
     <dynamics damping="1.0" friction="1.0"/>
-  </joint>`
-    <joint type="continuous" name="righ_wheel_hinge">
+  </joint>
+  <joint type="continuous" name="righ_wheel_hinge">
     <origin xyz="0 -0.15 0" rpy="0 0 0"/>
     <child link="right_wheel"/>

Commit message: [FEAT] Add colors to robot

File: catkin_ws/src/go_chase_it/urdf/my_robot.xacro (robot description, xacro)
@@ -175,3 +175,15 @@
     <dynamics damping="1.0" friction="1.0"/>
   </joint>
+  <gazebo reference="left_wheel">
+    <material>Gazebo/Green</material>
+  </gazebo>
+  <gazebo reference="right_wheel">
+    <material>Gazebo/Green</material>
+  </gazebo>
+  <gazebo reference="camera">
+    <material>Gazebo/Red</material>
+  </gazebo>
+  <gazebo reference="chassis">
+    <material>Gazebo/Blue</material>
+  </gazebo>
 </robot>

Commit message: [FIX] Correct caster wheel visual

File: catkin_ws/src/go_chase_it/urdf/my_robot.xacro (robot description, xacro)
@@ -50,5 +50,5 @@
     </collision>
     <visual name='front_caster_visual'>
-      <origin xyz="0.15 0 -0.5" rpy=" 0 1.5707 1.5707"/>
+      <origin xyz="0.15 0 -0.05" rpy=" 0 0 0"/>
       <geometry>
         <sphere radius="0.05"/>
@@ -168,5 +168,5 @@
     <dynamics damping="1.0" friction="1.0"/>
   </joint>
-  <joint type="continuous" name="righ_wheel_hinge">
+  <joint type="continuous" name="right_wheel_hinge">
     <origin xyz="0 -0.15 0" rpy="0 0 0"/>
     <child link="right_wheel"/>

Commit message: [FEAT] Make robot four wheeled

File: catkin_ws/src/go_chase_it/urdf/my_robot.xacro (robot description, xacro)
@@ -1,190 +1,229 @@
-<?xml version='1.0'?>
+<?xml version="1.0"?>
 <robot name="my_robot" xmlns:xacro="http://www.ros.org/wiki/xacro">
-<xacro:include filename="$(find go_chase_it)/urdf/my_robot.gazebo" />
-  <link name="robot_footprint"></link>
-  <joint name="robot_footprint_joint" type="fixed">
-    <origin xyz="0 0 0" rpy="0 0 0" />
-    <parent link="robot_footprint"/>
-    <child link="chassis" />
-  </joint>
-  <link name='chassis'>
-    <pose>0 0 0.1 0 0 0</pose>
-    <inertial>
-      <mass value="15.0"/>
-      <origin xyz="0.0 0 0" rpy=" 0 0 0"/>
-      <inertia
-          ixx="0.1" ixy="0" ixz="0"
-          iyy="0.1" iyz="0"
-          izz="0.1"
-      />
-    </inertial>
-    <collision name='collision'>
-      <origin xyz="0 0 0" rpy=" 0 0 0"/>
-      <geometry>
-        <box size=".4 .2 .1"/>
-      </geometry>
-    </collision>
-    <visual name='chassis_visual'>
-      <origin xyz="0 0 0" rpy=" 0 0 0"/>
-      <geometry>
-        <box size=".4 .2 .1"/>
-      </geometry>
-    </visual>
-    <collision name='back_caster_collision'>
-      <origin xyz="-0.15 0 -0.05" rpy=" 0 0 0"/>
-      <geometry>
-        <sphere radius="0.0499"/>
-      </geometry>
-    </collision>
-    <visual name='back_caster_visual'>
-      <origin xyz="-0.15 0 -0.05" rpy=" 0 0 0"/>
-      <geometry>
-        <sphere radius="0.05"/>
-      </geometry>
-    </visual>
-    <collision name='front_caster_collision'>
-      <origin xyz="0.15 0 -0.05" rpy=" 0 0 0"/>
-      <geometry>
-        <sphere radius="0.0499"/>
-      </geometry>
-    </collision>
-    <visual name='front_caster_visual'>
-      <origin xyz="0.15 0 -0.05" rpy=" 0 0 0"/>
-      <geometry>
-        <sphere radius="0.05"/>
-      </geometry>
-    </visual>
-  </link>
-  <link name= 'left_wheel'>
-    <visual>
-      <origin xyz="-0.0 0 0" rpy=" 0 1.5707 1.5707"/>
-      <geometry>
-        <cylinder radius="0.1" length="0.05"/>
-      </geometry>
-    </visual>
-    <collision>
-      <origin xyz="-0.0 0 0" rpy=" 0 1.5707 1.5707"/>
-      <geometry>
-        <cylinder radius="0.1" length="0.05"/>
-      </geometry>
-    </collision>
-    <inertial>
-      <mass value="5.0"/>
-      <origin xyz="0.0 0 0" rpy=" 0 1.5707 1.5707"/>
-      <inertia
-          ixx="0.1" ixy="0" ixz="0"
-          iyy="0.1" iyz="0"
-          izz="0.1"
-      />
-     </inertial>
-  </link>
-  <link name= 'right_wheel'>
-    <visual>
-      <origin xyz="-0.0 0 0" rpy=" 0 1.5707 1.5707"/>
-      <geometry>
-        <cylinder radius="0.1" length="0.05"/>
-      </geometry>
-    </visual>
-    <collision>
-      <origin xyz="-0.0 0 0" rpy=" 0 1.5707 1.5707"/>
-      <geometry>
-        <cylinder radius="0.1" length="0.05"/>
-      </geometry>
-    </collision>
-    <inertial>
-      <mass value="5.0"/>
-      <origin xyz="0.0 0 0" rpy=" 0 1.5707 1.5707"/>
-      <inertia
-          ixx="0.1" ixy="0" ixz="0"
-          iyy="0.1" iyz="0"
-          izz="0.1"
-      />
-    </inertial>
-  </link>
-  <link name='camera'>
-    <visual>
-      <origin xyz="-0.0 0 0" rpy=" 0 0 0"/>
-      <geometry>
-        <box size="0.05 0.05 0.05"/>
-      </geometry>
-    </visual>
-     <collision>
-      <origin xyz="-0.0 0 0" rpy=" 0 0 0"/>
-      <geometry>
-        <box size="0.05 0.05 0.05"/>
-      </geometry>
-    </collision>
-    <inertial>
-      <mass value="0.1"/>
-      <origin xyz="0.0 0 0" rpy=" 0 0 0"/>
-      <inertia
-          ixx="1e-6" ixy="0" ixz="0"
-          iyy="1e-6" iyz="0"
-          izz="1e-6"
-      />
-    </inertial>
-  </link>
-<link name='hokuyo'>
-    <visual>
-      <origin xyz="-0.0 0 0" rpy=" 0 0 0"/>
-      <geometry>
-        <mesh filename="package://go_chase_it/meshes/hokuyo.dae"/>
-      </geometry>
-    </visual>
-    <collision>
-      <origin xyz="-0.0 0 0" rpy=" 0 0 0"/>
-      <geometry>
-        <box size="0.01 0.01 0.01"/>
-      </geometry>
-    </collision>
-    <inertial>
-      <mass value="1e-5"/>
-      <origin xyz="0.0 0 0" rpy=" 0 0 0"/>
-      <inertia
-          ixx="1e-6" ixy="0" ixz="0"
-          iyy="1e-6" iyz="0"
-          izz="1e-6"
-      />
-    </inertial>
-  </link>
-  <joint type="fixed" name="camera_joint">
-    <origin xyz="0.2 0 0" rpy="0 0 0"/>
-    <child link="camera"/>
-    <parent link="chassis"/>
-    <axis xyz="0 1 0" rpy="0 0 0"/>
-  </joint>
-  <joint type="fixed" name="hokuyo">
-    <origin xyz="0.15 0 0.1" rpy="0 0 0"/>
-    <child link="hokuyo"/>
-    <parent link="chassis"/>
-    <axis xyz="0 1 0" rpy="0 0 0"/>
-  </joint>
-  <joint type="continuous" name="left_wheel_hinge">
-    <origin xyz="0 0.15 0" rpy="0 0 0"/>
-    <child link="left_wheel"/>
-    <parent link="chassis"/>
-    <axis xyz="0 1 0" rpy="0 0 0"/>
-    <limit effort="10000" velocity="1000"/>
-    <dynamics damping="1.0" friction="1.0"/>
-  </joint>
-  <joint type="continuous" name="right_wheel_hinge">
-    <origin xyz="0 -0.15 0" rpy="0 0 0"/>
-    <child link="right_wheel"/>
-    <parent link="chassis"/>
-    <axis xyz="0 1 0" rpy="0 0 0"/>
-    <limit effort="10000" velocity="1000"/>
-    <dynamics damping="1.0" friction="1.0"/>
-  </joint>
-  <gazebo reference="left_wheel">
-    <material>Gazebo/Green</material>
-  </gazebo>
-  <gazebo reference="right_wheel">
-    <material>Gazebo/Green</material>
-  </gazebo>
-  <gazebo reference="camera">
-    <material>Gazebo/Red</material>
-  </gazebo>
-  <gazebo reference="chassis">
-    <material>Gazebo/Blue</material>
-  </gazebo>
+	<include filename="$(find go_chase_it)/urdf/my_robot.gazebo" />
+	<!--  Footprint -->
+	<link name="robot_footprint">
+	</link>
+	<joint name="robot_footprint_joint" type="fixed">
+		<origin xyz="0 0 0" rpy="0 0 0" />
+		<parent link="robot_footprint" />
+		<child link="chassis" />
+	</joint>
+	<!-- Chassis -->
+	<link name="chassis">
+		<pose>
+			0 0 0.1 0 0 0
+		</pose>
+		<inertial>
+			<mass value="15.0" />
+			<origin xyz="0.0 0 0" rpy=" 0 0 0" />
+			<inertia ixx="0.1" ixy="0" ixz="0" iyy="0.1" iyz="0" izz="0.1" />
+		</inertial>
+		<collision name="collision">
+			<origin xyz="0 0 0" rpy=" 0 0 0" />
+			<geometry>
+				<box size=".8 .2 .1" />
+			</geometry>
+		</collision>
+		<visual name="chassis_visual">
+			<origin xyz="0 0 0" rpy=" 0 0 0" />
+			<geometry>
+				<box size=".8 .2 .1" />
+			</geometry>
+		</visual>
+	</link>
+	<gazebo reference="chassis">
+		<material>
+			Gazebo/Blue
+		</material>
+	</gazebo>
+	<!-- Right Front Wheel -->
+	<link name="front_right_wheel">
+		<visual>
+			<origin xyz="0.35 0 0" rpy=" 0 1.5707 1.5707" />
+			<geometry>
+				<cylinder radius="0.1" length="0.05" />
+			</geometry>
+		</visual>
+		<collision>
+			<origin xyz="0.35 0 0" rpy=" 0 1.5707 1.5707" />
+			<geometry>
+				<cylinder radius="0.1" length="0.05" />
+			</geometry>
+		</collision>
+		<inertial>
+			<mass value="5.0" />
+			<origin xyz="0.35 0 0" rpy=" 0 1.5707 1.5707" />
+			<inertia ixx="0.1" ixy="0" ixz="0" iyy="0.1" iyz="0" izz="0.1" />
+		</inertial>
+	</link>
+	<joint type="continuous" name="front_right_wheel_hinge">
+		<origin xyz="0.35 -0.15 0" rpy="0 0 0" />
+		<child link="front_right_wheel" />
+		<parent link="chassis" />
+		<axis xyz="0 1 0" rpy="0 0 0" />
+		<limit effort="10000" velocity="1000" />
+		<dynamics damping="1.0" friction="1.0" />
+	</joint>
+	<gazebo reference="front_right_wheel">
+		<material>
+			Gazebo/Green
+		</material>
+	</gazebo>
+	<!-- Left Front Wheel -->
+	<link name="front_left_wheel">
+		<visual>
+			<origin xyz="0.35 0 0" rpy=" 0 1.5707 1.5707" />
+			<geometry>
+				<cylinder radius="0.1" length="0.05" />
+			</geometry>
+		</visual>
+		<collision>
+			<origin xyz="0.35 0 0" rpy=" 0 1.5707 1.5707" />
+			<geometry>
+				<cylinder radius="0.1" length="0.05" />
+			</geometry>
+		</collision>
+		<inertial>
+			<mass value="5.0" />
+			<origin xyz="0.35 0 0" rpy=" 0 1.5707 1.5707" />
+			<inertia ixx="0.1" ixy="0" ixz="0" iyy="0.1" iyz="0" izz="0.1" />
+		</inertial>
+	</link>
+	<joint type="continuous" name="front_left_wheel_hinge">
+		<origin xyz="0.35 0.15 0" rpy="0 0 0" />
+		<child link="front_left_wheel" />
+		<parent link="chassis" />
+		<axis xyz="0 1 0" rpy="0 0 0" />
+		<limit effort="10000" velocity="1000" />
+		<dynamics damping="1.0" friction="1.0" />
+	</joint>
+	<gazebo reference="front_left_wheel">
+		<material>
+			Gazebo/Green
+		</material>
+	</gazebo>
+	<!-- Back Left Wheel -->
+	<link name="back_left_wheel">
+		<visual>
+			<origin xyz="-0.35 0 0" rpy=" 0 1.5707 1.5707" />
+			<geometry>
+				<cylinder radius="0.1" length="0.05" />
+			</geometry>
+		</visual>
+		<collision>
+			<origin xyz="-0.35 0 0" rpy=" 0 1.5707 1.5707" />
+			<geometry>
+				<cylinder radius="0.1" length="0.05" />
+			</geometry>
+		</collision>
+		<inertial>
+			<mass value="5.0" />
+			<origin xyz="-0.35 0 0" rpy=" 0 1.5707 1.5707" />
+			<inertia ixx="0.1" ixy="0" ixz="0" iyy="0.1" iyz="0" izz="0.1" />
+		</inertial>
+	</link>
+	<joint type="continuous" name="back_left_wheel_hinge">
+		<origin xyz="-0.35 0.15 0" rpy="0 0 0" />
+		<child link="back_left_wheel" />
+		<parent link="chassis" />
+		<axis xyz="0 1 0" rpy="0 0 0" />
+		<limit effort="10000" velocity="1000" />
+		<dynamics damping="1.0" friction="1.0" />
+	</joint>
+	<gazebo reference="back_left_wheel">
+		<material>
+			Gazebo/Green
+		</material>
+	</gazebo>
+	<!-- Back Right Wheel -->
+	<link name="back_right_wheel">
+		<visual>
+			<origin xyz="-0.35 0 0" rpy=" 0 1.5707 1.5707" />
+			<geometry>
+				<cylinder radius="0.1" length="0.05" />
+			</geometry>
+		</visual>
+		<collision>
+			<origin xyz="-0.35 0 0" rpy=" 0 1.5707 1.5707" />
+			<geometry>
+				<cylinder radius="0.1" length="0.05" />
+			</geometry>
+		</collision>
+		<inertial>
+			<mass value="5.0" />
+			<origin xyz="-0.35 0 0" rpy=" 0 1.5707 1.5707" />
+			<inertia ixx="0.1" ixy="0" ixz="0" iyy="0.1" iyz="0" izz="0.1" />
+		</inertial>
+	</link>
+	<joint type="continuous" name="back_right_wheel_hinge">
+		<origin xyz="-0.35 -0.15 0" rpy="0 0 0" />
+		<child link="back_right_wheel" />
+		<parent link="chassis" />
+		<axis xyz="0 1 0" rpy="0 0 0" />
+		<limit effort="10000" velocity="1000" />
+		<dynamics damping="1.0" friction="1.0" />
+	</joint>
+	<gazebo reference="back_right_wheel">
+		<material>
+			Gazebo/Green
+		</material>
+	</gazebo>
+	<!-- Camera -->
+	<link name="camera">
+		<visual>
+			<origin xyz="-0.0 0 0" rpy=" 0 0 0" />
+			<geometry>
+				<box size="0.05 0.05 0.05" />
+			</geometry>
+		</visual>
+		<collision>
+			<origin xyz="-0.0 0 0" rpy=" 0 0 0" />
+			<geometry>
+				<box size="0.05 0.05 0.05" />
+			</geometry>
+		</collision>
+		<inertial>
+			<mass value="0.1" />
+			<origin xyz="0.0 0 0" rpy=" 0 0 0" />
+			<inertia ixx="1e-6" ixy="0" ixz="0" iyy="1e-6" iyz="0" izz="1e-6" />
+		</inertial>
+	</link>
+	<joint type="fixed" name="camera_joint">
+		<origin xyz="0.4 0 0" rpy="0 0 0" />
+		<child link="camera" />
+		<parent link="chassis" />
+		<axis xyz="0 1 0" rpy="0 0 0" />
+	</joint>
+	<gazebo reference="camera">
+		<material>
+			Gazebo/Red
+		</material>
+	</gazebo>
+	<!-- LIDAR -->
+	<link name="hokuyo">
+		<visual>
+			<origin xyz="-0.0 0 0" rpy=" 0 0 0" />
+			<geometry>
+				<mesh filename="package://go_chase_it/meshes/hokuyo.dae" />
+			</geometry>
+		</visual>
+		<collision>
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
Commit message: [FIX] Correct robot dimensions and joints

File: catkin_ws/src/go_chase_it/urdf/my_robot.xacro (robot description, xacro)
@@ -23,5 +23,5 @@
 			<origin xyz="0 0 0" rpy=" 0 0 0" />
 			<geometry>
-				<box size=".8 .2 .1" />
+				<box size=".8 .5 .1" />
 			</geometry>
 		</collision>
@@ -29,5 +29,5 @@
 			<origin xyz="0 0 0" rpy=" 0 0 0" />
 			<geometry>
-				<box size=".8 .2 .1" />
+				<box size=".8 .5 .1" />
 			</geometry>
 		</visual>
@@ -41,23 +41,23 @@
 	<link name="front_right_wheel">
 		<visual>
-			<origin xyz="0.35 0 0" rpy=" 0 1.5707 1.5707" />
-			<geometry>
-				<cylinder radius="0.1" length="0.05" />
-			</geometry>
-		</visual>
-		<collision>
-			<origin xyz="0.35 0 0" rpy=" 0 1.5707 1.5707" />
-			<geometry>
-				<cylinder radius="0.1" length="0.05" />
-			</geometry>
-		</collision>
-		<inertial>
-			<mass value="5.0" />
-			<origin xyz="0.35 0 0" rpy=" 0 1.5707 1.5707" />
+			<origin xyz="0 0 0" rpy=" 0 1.5707 1.5707" />
+			<geometry>
+				<cylinder radius="0.1" length="0.05" />
+			</geometry>
+		</visual>
+		<collision>
+			<origin xyz="0 0 0" rpy=" 0 1.5707 1.5707" />
+			<geometry>
+				<cylinder radius="0.1" length="0.05" />
+			</geometry>
+		</collision>
+		<inertial>
+			<mass value="5.0" />
+			<origin xyz="0 0 0" rpy=" 0 1.5707 1.5707" />
 			<inertia ixx="0.1" ixy="0" ixz="0" iyy="0.1" iyz="0" izz="0.1" />
 		</inertial>
 	</link>
 	<joint type="continuous" name="front_right_wheel_hinge">
-		<origin xyz="0.35 -0.15 0" rpy="0 0 0" />
+		<origin xyz="0.2 -0.3 0" rpy="0 0 0" />
 		<child link="front_right_wheel" />
 		<parent link="chassis" />
@@ -68,5 +68,5 @@
 	<gazebo reference="front_right_wheel">
 		<material>
-			Gazebo/Green
+			Gazebo/Blue
 		</material>
 	</gazebo>
@@ -74,23 +74,23 @@
 	<link name="front_left_wheel">
 		<visual>
-			<origin xyz="0.35 0 0" rpy=" 0 1.5707 1.5707" />
-			<geometry>
-				<cylinder radius="0.1" length="0.05" />
-			</geometry>
-		</visual>
-		<collision>
-			<origin xyz="0.35 0 0" rpy=" 0 1.5707 1.5707" />
-			<geometry>
-				<cylinder radius="0.1" length="0.05" />
-			</geometry>
-		</collision>
-		<inertial>
-			<mass value="5.0" />
-			<origin xyz="0.35 0 0" rpy=" 0 1.5707 1.5707" />
+			<origin xyz="0 0 0" rpy=" 0 1.5707 1.5707" />
+			<geometry>
+				<cylinder radius="0.1" length="0.05" />
+			</geometry>
+		</visual>
+		<collision>
+			<origin xyz="0 0 0" rpy=" 0 1.5707 1.5707" />
+			<geometry>
+				<cylinder radius="0.1" length="0.05" />
+			</geometry>
+		</collision>
+		<inertial>
+			<mass value="5.0" />
+			<origin xyz="0 0 0" rpy=" 0 1.5707 1.5707" />
 			<inertia ixx="0.1" ixy="0" ixz="0" iyy="0.1" iyz="0" izz="0.1" />
 		</inertial>
 	</link>
 	<joint type="continuous" name="front_left_wheel_hinge">
-		<origin xyz="0.35 0.15 0" rpy="0 0 0" />
+		<origin xyz="0.2 0.3 0" rpy="0 0 0" />
 		<child link="front_left_wheel" />
 		<parent link="chassis" />
@@ -101,5 +101,5 @@
 	<gazebo reference="front_left_wheel">
 		<material>
-			Gazebo/Green
+			Gazebo/Blue
 		</material>
 	</gazebo>
@@ -107,23 +107,23 @@
 	<link name="back_left_wheel">
 		<visual>
-			<origin xyz="-0.35 0 0" rpy=" 0 1.5707 1.5707" />
-			<geometry>
-				<cylinder radius="0.1" length="0.05" />
-			</geometry>
-		</visual>
-		<collision>
-			<origin xyz="-0.35 0 0" rpy=" 0 1.5707 1.5707" />
-			<geometry>
-				<cylinder radius="0.1" length="0.05" />
-			</geometry>
-		</collision>
-		<inertial>
-			<mass value="5.0" />
-			<origin xyz="-0.35 0 0" rpy=" 0 1.5707 1.5707" />
+			<origin xyz="-0 0 0" rpy=" 0 1.5707 1.5707" />
+			<geometry>
+				<cylinder radius="0.1" length="0.05" />
+			</geometry>
+		</visual>
+		<collision>
+			<origin xyz="-0 0 0" rpy=" 0 1.5707 1.5707" />
+			<geometry>
+				<cylinder radius="0.1" length="0.05" />
+			</geometry>
+		</collision>
+		<inertial>
+			<mass value="5.0" />
+			<origin xyz="-0 0 0" rpy=" 0 1.5707 1.5707" />
 			<inertia ixx="0.1" ixy="0" ixz="0" iyy="0.1" iyz="0" izz="0.1" />
 		</inertial>
 	</link>
 	<joint type="continuous" name="back_left_wheel_hinge">
-		<origin xyz="-0.35 0.15 0" rpy="0 0 0" />
+		<origin xyz="-0.2 0.3 0" rpy="0 0 0" />
 		<child link="back_left_wheel" />
 		<parent link="chassis" />
@@ -134,5 +134,5 @@
 	<gazebo reference="back_left_wheel">
 		<material>
-			Gazebo/Green
+			Gazebo/Blue
 		</material>
 	</gazebo>
@@ -140,23 +140,23 @@
 	<link name="back_right_wheel">
 		<visual>
-			<origin xyz="-0.35 0 0" rpy=" 0 1.5707 1.5707" />
-			<geometry>
-				<cylinder radius="0.1" length="0.05" />
-			</geometry>
-		</visual>
-		<collision>
-			<origin xyz="-0.35 0 0" rpy=" 0 1.5707 1.5707" />
-			<geometry>
-				<cylinder radius="0.1" length="0.05" />
-			</geometry>
-		</collision>
-		<inertial>
-			<mass value="5.0" />
-			<origin xyz="-0.35 0 0" rpy=" 0 1.5707 1.5707" />
+			<origin xyz="-0 0 0" rpy=" 0 1.5707 1.5707" />
+			<geometry>
+				<cylinder radius="0.1" length="0.05" />
+			</geometry>
+		</visual>
+		<collision>
+			<origin xyz="-0 0 0" rpy=" 0 1.5707 1.5707" />
+			<geometry>
+				<cylinder radius="0.1" length="0.05" />
+			</geometry>
+		</collision>
+		<inertial>
+			<mass value="5.0" />
+			<origin xyz="-0 0 0" rpy=" 0 1.5707 1.5707" />
 			<inertia ixx="0.1" ixy="0" ixz="0" iyy="0.1" iyz="0" izz="0.1" />
 		</inertial>
 	</link>
 	<joint type="continuous" name="back_right_wheel_hinge">
-		<origin xyz="-0.35 -0.15 0" rpy="0 0 0" />
+		<origin xyz="-0.2 -0.3 0" rpy="0 0 0" />
 		<child link="back_right_wheel" />
 		<parent link="chassis" />
@@ -167,5 +167,5 @@
 	<gazebo reference="back_right_wheel">
 		<material>
-			Gazebo/Green
+			Gazebo/Blue
 		</material>
 	</gazebo>
